File: 01-loeterli-board/loeterli-board/loeterli-board.sch (KiCad schematic (older format))
At the start: 96 parts, among them J1 RPC1-12RB-6P, J2 Conn_01x01, J3 Conn_01x04, J5 Screw_Terminal_01x03, Q1 PSMN5R2-60YL, SW1 SW_Push, SW2 SW_Push, SW3 SW_Push, SW4 SW_Push, U1 VOM1271T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

Commit message: layout changes
Parts:
- C19, C20, C21, C22, C23: footprint Capacitor_SMD:C_1206_3216Metric -> Capacitor_SMD:C_0603_1608Metric
Changed lines of the file:
@@
 EESchema Schematic File Version 4
-LIBS:loeterli-board-cache
 EELAYER 30 0
 EELAYER END
@@
 F 0 "C22" H 2765 2946 50  0000 L CNN
 F 1 "C" H 2765 2855 50  0000 L CNN
-F 2 "Capacitor_SMD:C_1206_3216Metric" H 2688 2750 50  0001 C CNN
+F 2 "Capacitor_SMD:C_0603_1608Metric" H 2688 2750 50  0001 C CNN
 F 3 "~" H 2650 2900 50  0001 C CNN
 	1    2650 2900
@@
 F 0 "C20" H 1365 5896 50  0000 L CNN
 F 1 "C" H 1365 5805 50  0000 L CNN
-F 2 "Capacitor_SMD:C_1206_3216Metric" H 1288 5700 50  0001 C CNN
+F 2 "Capacitor_SMD:C_0603_1608Metric" H 1288 5700 50  0001 C CNN
 F 3 "~" H 1250 5850 50  0001 C CNN
 	1    1250 5850
@@
 F 0 "C21" H 1365 7246 50  0000 L CNN
 F 1 "C" H 1365 7155 50  0000 L CNN
-F 2 "Capacitor_SMD:C_1206_3216Metric" H 1288 7050 50  0001 C CNN
+F 2 "Capacitor_SMD:C_0603_1608Metric" H 1288 7050 50  0001 C CNN
 F 3 "~" H 1250 7200 50  0001 C CNN
 	1    1250 7200
@@
 F 0 "C19" H 1365 4596 50  0000 L CNN
 F 1 "C" H 1365 4505 50  0000 L CNN
-F 2 "Capacitor_SMD:C_1206_3216Metric" H 1288 4400 50  0001 C CNN
+F 2 "Capacitor_SMD:C_0603_1608Metric" H 1288 4400 50  0001 C CNN
 F 3 "~" H 1250 4550 50  0001 C CNN
 	1    1250 4550
@@
 F 0 "C23" H 3365 5946 50  0000 L CNN
 F 1 "C" H 3365 5855 50  0000 L CNN
-F 2 "Capacitor_SMD:C_1206_3216Metric" H 3288 5750 50  0001 C CNN
+F 2 "Capacitor_SMD:C_0603_1608Metric" H 3288 5750 50  0001 C CNN
 F 3 "~" H 3250 5900 50  0001 C CNN
 	1    3250 5900
